File: pcb/MacroBoard.kicad_pcb (KiCad board)
At the start: 2 copper layers, 61 x 86.4 mm, 9 parts, among them U1 Pico, U2 PEC12R-4025F-S0024

Commit message: Added name in pcb
Other:
- board text added: "macro-board v-1.0.0 Designed by Rithul Kamesh"
Changed lines of the file:
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@@
       (effects (font (size 0.8 0.8) (thickness 0.15)))
-    )
-    (fp_text user "Copper Keepouts shown on Dwgs layer" (at 0.1 -30.2 90) (layer "Cmts.User")
-      (effects (font (size 1 1) (thickness 0.15)))
     )
     (fp_text user "${REFERENCE}" (at 0 0 90) (layer "F.Fab")
@@
   (gr_arc (start 106.68 137.16) (mid 104.883949 136.416051) (end 104.14 134.62) (layer "Edge.Cuts") (width 0.1))
   (gr_line (start 106.68 137.16) (end 162.56 137.16) (layer "Edge.Cuts") (width 0.1))
+  (gr_text "macro-board v-1.0.0\nDesigned by Rithul Kamesh\n" (at 139.7 68.58) (layer "B.Cu")
+    (effects (font (size 1.5 1.5) (thickness 0.3)) (justify mirror))
+  )
   (segment (start 132.64 93.42) (end 141.62 93.42) (width 0.25) (layer "F.Cu") (net 19))
   (segment (start 123.19 95.25) (end 124.46 96.52) (width 0.25) (layer "F.Cu") (net 19))

Commit message: Archive Commit
Parts:
- added REF**: MountingHole_2.1mm, MountingHole:MountingHole_2.1mm, F.Cu at (162.6, 53.3)
- added REF**: MountingHole_2.1mm, MountingHole:MountingHole_2.1mm, F.Cu at (162.6, 137.2)
- added REF**: MountingHole_2.1mm, MountingHole:MountingHole_2.1mm, F.Cu at (106.7, 53.3)
- added REF**: MountingHole_2.1mm, MountingHole:MountingHole_2.1mm, F.Cu at (106.7, 137.2)
Other:
- board size 61 x 86.4 mm -> 61 x 89.6 mm
Changed lines of the file:
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@@
     )
     (pad_to_mask_clearance 0)
+    (grid_origin 134.62 139.7)
     (pcbplotparams
       (layerselection 0x00010fc_ffffffff)
@@
   (net 54 "Col2")
   (net 55 "Col3")
+  (footprint "MountingHole:MountingHole_2.1mm" (layer "F.Cu")
+    (at 162.56 53.34)
+    (descr "Mounting Hole 2.1mm, no annular")
+    (tags "mounting hole 2.1mm no annular")
+    (attr exclude_from_pos_files exclude_from_bom)
+    (fp_text reference "REF**" (at 0 -3.2) (layer "F.SilkS")
+      (effects (font (size 1 1) (thickness 0.15)))
+    )
+    (fp_text value "MountingHole_2.1mm" (at 0 3.2) (layer "F.Fab")
+      (effects (font (size 1 1) (thickness 0.15)))
+    )
+    (fp_text user "${REFERENCE}" (at 0 0) (layer "F.Fab")
+      (effects (font (size 1 1) (thickness 0.15)))
+    )
+    (fp_circle (center 0 0) (end 2.1 0) (layer "Cmts.User") (width 0.15) (fill none))
+    (fp_circle (center 0 0) (end 2.35 0) (layer "F.CrtYd") (width 0.05) (fill none))
+    (pad "" np_thru_hole circle (at 0 0) (size 2.1 2.1) (drill 2.1) (layers *.Cu *.Mask))
+  )
   (footprint "MX1A11NW:MX1A11NW" (layer "F.Cu")
     (at 151.13 124.46)
@@
       (rotate (xyz 0 0 0))
     )
+  )
+  (footprint "MountingHole:MountingHole_2.1mm" (layer "F.Cu")
+    (at 162.56 137.16)
+    (descr "Mounting Hole 2.1mm, no annular")
+    (tags "mounting hole 2.1mm no annular")
+    (attr exclude_from_pos_files exclude_from_bom)
+    (fp_text reference "REF**" (at 12.7 -2.36) (layer "F.SilkS")
+      (effects (font (size 1 1) (thickness 0.15)))
+    )
+    (fp_text value "MountingHole_2.1mm" (at 0 3.2) (layer "F.Fab")
+      (effects (font (size 1 1) (thickness 0.15)))
+    )
+    (fp_text user "${REFERENCE}" (at 0 0) (layer "F.Fab")
+      (effects (font (size 1 1) (thickness 0.15)))
+    )
+    (fp_circle (center 0 0) (end 2.1 0) (layer "Cmts.User") (width 0.15) (fill none))
+    (fp_circle (center 0 0) (end 2.35 0) (layer "F.CrtYd") (width 0.05) (fill none))
+    (pad "" np_thru_hole circle (at 0 0) (size 2.1 2.1) (drill 2.1) (layers *.Cu *.Mask))
   )
   (footprint "MCU_RaspberryPi_and_Boards:RPi_Pico_SMD_TH" (layer "F.Cu")
@@
     (pad "43" smd rect locked (at 2.54 23.9) (size 3.5 1.7) (drill (offset -0.9 0)) (layers "F.Cu" "F.Mask")
       (net 37 "unconnected-(U1-Pad43)") (pinfunction "SWDIO") (pintype "bidirectional"))
+  )
+  (footprint "MountingHole:MountingHole_2.1mm" (layer "F.Cu")
+    (at 106.68 53.34)
+    (descr "Mounting Hole 2.1mm, no annular")
+    (tags "mounting hole 2.1mm no annular")
+    (attr exclude_from_pos_files exclude_from_bom)
+    (fp_text reference "REF**" (at 0 -3.2) (layer "F.SilkS")
+      (effects (font (size 1 1) (thickness 0.15)))
+    )
+    (fp_text value "MountingHole_2.1mm" (at 0 3.2) (layer "F.Fab")
+      (effects (font (size 1 1) (thickness 0.15)))
+    )
+    (fp_text user "${REFERENCE}" (at 0 0) (layer "F.Fab")
+      (effects (font (size 1 1) (thickness 0.15)))
+    )
+    (fp_circle (center 0 0) (end 2.1 0) (layer "Cmts.User") (width 0.15) (fill none))
+    (fp_circle (center 0 0) (end 2.35 0) (layer "F.CrtYd") (width 0.05) (fill none))
+    (pad "" np_thru_hole circle (at 0 0) (size 2.1 2.1) (drill 2.1) (layers *.Cu *.Mask))
+  )
+  (footprint "MountingHole:MountingHole_2.1mm" (layer "F.Cu")
+    (at 106.68 137.16)
+    (descr "Mounting Hole 2.1mm, no annular")
+    (tags "mounting hole 2.1mm no annular")
+    (attr exclude_from_pos_files exclude_from_bom)
+    (fp_text reference "REF**" (at -17.78 -7.62) (layer "F.SilkS")
+      (effects (font (size 1 1) (thickness 0.15)))
+    )
+    (fp_text value "MountingHole_2.1mm" (at 0 3.2) (layer "F.Fab")
+      (effects (font (size 1 1) (thickness 0.15)))
+    )
+    (fp_text user "${REFERENCE}" (at 0 0) (layer "F.Fab")
+      (effects (font (size 1 1) (thickness 0.15)))
+    )
+    (fp_circle (center 0 0) (end 2.1 0) (layer "Cmts.User") (width 0.15) (fill none))
+    (fp_circle (center 0 0) (end 2.35 0) (layer "F.CrtYd") (width 0.05) (fill none))
+    (pad "" np_thru_hole circle (at 0 0) (size 2.1 2.1) (drill 2.1) (layers *.Cu *.Mask))
   )
   (footprint "MX1A11NW:MX1A11NW" (layer "F.Cu")
@@
       ) (layer "B.SilkS") (width 0) (fill solid))
   )
-  (gr_arc (start 165.1 134.62) (mid 164.356051 136.416051) (end 162.56 137.16) (layer "Edge.Cuts") (width 0.1))
-  (gr_line (start 104.14 53.34) (end 104.14 134.62) (layer "Edge.Cuts") (width 0.1))
+  (gr_arc (start 165.1 137.903949) (mid 164.356051 139.7) (end 162.56 140.443949) (layer "Edge.Cuts") (width 0.1))
+  (gr_line (start 104.14 53.34) (end 104.14 137.903949) (layer "Edge.Cuts") (width 0.1))
   (gr_line (start 106.68 50.8) (end 162.56 50.8) (layer "Edge.Cuts") (width 0.1))
   (gr_arc (start 104.14 53.34) (mid 104.883949 51.543949) (end 106.68 50.8) (layer "Edge.Cuts") (width 0.1))
-  (gr_line (start 165.1 134.62) (end 165.1 53.34) (layer "Edge.Cuts") (width 0.1))
+  (gr_line (start 165.1 137.903949) (end 165.1 53.34) (layer "Edge.Cuts") (width 0.1))
   (gr_arc (start 162.56 50.8) (mid 164.356051 51.543949) (end 165.1 53.34) (layer "Edge.Cuts") (width 0.1))
-  (gr_arc (start 106.68 137.16) (mid 104.883949 136.416051) (end 104.14 134.62) (layer "Edge.Cuts") (width 0.1))
-  (gr_line (start 106.68 137.16) (end 162.56 137.16) (layer "Edge.Cuts") (width 0.1))
+  (gr_arc (start 106.68 140.443949) (mid 104.883949 139.7) (end 104.14 137.903949) (layer "Edge.Cuts") (width 0.1))
+  (gr_line (start 106.68 140.443949) (end 162.56 140.443949) (layer "Edge.Cuts") (width 0.1))
   (gr_text "macro-board v-1.0.0\nDesigned by Rithul Kamesh\n" (at 139.7 68.58) (layer "B.Cu")
     (effects (font (size 1.5 1.5) (thickness 0.3)) (justify mirror))
@@
     (connect_pads (clearance 0.508))
     (min_thickness 0.254) (filled_areas_thickness no)
-    (fill yes (thermal_gap 0.508) (thermal_bridge_width 0.508))
+    (fill (thermal_gap 0.508) (thermal_bridge_width 0.508))
     (polygon
       (pts
-        (xy 165.1 137.16)
-        (xy 104.14 137.16)
-        (xy 104.14 50.8)
-        (xy 165.1 50.8)
+        (xy 165.1 139.7)
+        (xy 104.14 139.7)
+        (xy 104.14 53.34)
+        (xy 165.1 53.34)
       )
     )
